File: torque_motor_design.kicad_pcb (KiCad board)
At the start: 2 copper layers, 27.9 x 37 mm, 38 parts, among them U1 ATtiny85-20S, U2 OPAMP, U3 OPAMP, U4 L78L05_SO8

Commit message: Add:Version_1
Parts:
- RV1: footprint Potentiometer_SMD:Potentiometer_Bourns_3214W_Vertical -> Potentiometer_SMD:Potentiometer_Bourns_3224W_Vertical
Routing:
- net -V: track 115.4 -> 129.6 mm
Changed lines of the file:
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@@
       (drillshape 0)
       (scaleselection 1)
-      (outputdirectory "Component_Placement/")
+      (outputdirectory "Gerber Files/")
     )
   )
@@
     )
   )
-  (footprint "Potentiometer_SMD:Potentiometer_Bourns_3214W_Vertical" (layer "F.Cu")
+  (footprint "Potentiometer_SMD:Potentiometer_Bourns_3224W_Vertical" (layer "F.Cu")
     (at 185.5 42.3 180)
-    (descr "Potentiometer, vertical, Bourns 3214W, https://www.bourns.com/docs/Product-Datasheets/3214.pdf")
-    (tags "Potentiometer vertical Bourns 3214W")
-    (property "Sheetfile" "torque_motor_design.kicad_sch")
-    (property "Sheetname" "")
-    (attr smd)
-    (fp_text reference "RV1" (at 3.3 0.1 90 unlocked) (layer "F.SilkS")
-      (effects (font (size 0.225 0.15) (thickness 0.15)))
-    )
-    (fp_text value "1k" (at 0 3.5) (layer "F.Fab")
-      (effects (font (size 1 1) (thickness 0.15)))
-    )
-    (fp_text user "${REFERENCE}" (at 0.6 0) (layer "F.Fab")
+    (descr "Potentiometer, vertical, Bourns 3224W, https://www.bourns.com/docs/Product-Datasheets/3224.pdf")
+    (tags "Potentiometer vertical Bourns 3224W")
+    (property "Sheetfile" "torque_motor_design.kicad_sch")
+    (property "Sheetname" "")
+    (attr smd)
+    (fp_text reference "RV1" (at 2.89 0 180) (layer "F.SilkS")
+      (effects (font (size 0.15 0.15) (thickness 0.0375)))
+    )
+    (fp_text value "1k" (at 0 3.5 180) (layer "F.Fab")
+      (effects (font (size 1 1) (thickness 0.15)))
+    )
+    (fp_text user "${REFERENCE}" (at 0.6 0 180) (layer "F.Fab")
       (effects (font (size 0.6 0.6) (thickness 0.15)))
     )
-    (fp_line (start 2.52 -1.87) (end 2.52 1.87) (layer "F.SilkS") (width 0.12))
+    (fp_line (start 1.24 1.87) (end 2.52 1.87) (layer "F.SilkS") (width 0.12))
     (fp_line (start 2.14 -1.87) (end 2.52 -1.87) (layer "F.SilkS") (width 0.12))
     (fp_line (start -2.52 -1.87) (end -2.14 -1.87) (layer "F.SilkS") (width 0.12))
-    (fp_line (start 1.24 1.87) (end 2.52 1.87) (layer "F.SilkS") (width 0.12))
-    (fp_line (start -0.36 -1.87) (end 0.36 -1.87) (layer "F.SilkS") (width 0.12))
+    (fp_line (start 2.52 -1.87) (end 2.52 1.87) (layer "F.SilkS") (width 0.12))
     (fp_line (start -2.52 -1.87) (end -2.52 1.87) (layer "F.SilkS") (width 0.12))
     (fp_line (start -2.52 1.87) (end -1.24 1.87) (layer "F.SilkS") (width 0.12))
+    (fp_line (start -0.36 -1.87) (end 0.36 -1.87) (layer "F.SilkS") (width 0.12))
+    (fp_line (start 2.65 2.5) (end 2.65 -2.5) (layer "F.CrtYd") (width 0.05))
     (fp_line (start -2.65 -2.5) (end -2.65 2.5) (layer "F.CrtYd") (width 0.05))
     (fp_line (start -2.65 2.5) (end 2.65 2.5) (layer "F.CrtYd") (width 0.05))
-    (fp_line (start 2.65 2.5) (end 2.65 -2.5) (layer "F.CrtYd") (width 0.05))
     (fp_line (start 2.65 -2.5) (end -2.65 -2.5) (layer "F.CrtYd") (width 0.05))
+    (fp_line (start -2.4 -1.75) (end -2.4 1.75) (layer "F.Fab") (width 0.1))
+    (fp_line (start -1.2 1.393) (end -1.199 -0.092) (layer "F.Fab") (width 0.1))
     (fp_line (start 2.4 1.75) (end 2.4 -1.75) (layer "F.Fab") (width 0.1))
+    (fp_line (start 2.4 -1.75) (end -2.4 -1.75) (layer "F.Fab") (width 0.1))
     (fp_line (start -1.2 1.393) (end -1.199 -0.092) (layer "F.Fab") (width 0.1))
-    (fp_line (start 2.4 -1.75) (end -2.4 -1.75) (layer "F.Fab") (width 0.1))
-    (fp_line (start -2.4 -1.75) (end -2.4 1.75) (layer "F.Fab") (width 0.1))
     (fp_line (start -2.4 1.75) (end 2.4 1.75) (layer "F.Fab") (width 0.1))
-    (fp_line (start -1.2 1.393) (end -1.199 -0.092) (layer "F.Fab") (width 0.1))
     (fp_circle (center -1.2 0.65) (end -0.45 0.65) (layer "F.Fab") (width 0.1) (fill none))
     (pad "1" smd rect (at 1.25 -1.45 180) (size 1.3 1.6) (layers "F.Cu" "F.Paste" "F.Mask")
@@
     (pad "3" smd rect (at -1.25 -1.45 180) (size 1.3 1.6) (layers "F.Cu" "F.Paste" "F.Mask")
       (net 9 "Net-(R1-Pad2)") (pinfunction "3") (pintype "passive"))
-    (model "${KICAD6_3DMODEL_DIR}/Potentiometer_SMD.3dshapes/Potentiometer_Bourns_3214W_Vertical.wrl"
+    (model "${KICAD6_3DMODEL_DIR}/Potentiometer_SMD.3dshapes/Potentiometer_Bourns_3224W_Vertical.wrl"
       (offset (xyz 0 0 0))
       (scale (xyz 1 1 1))
@@
   )
   (segment (start 195.25 54.98) (end 194.953573 54.98) (width 0.4) (layer "F.Cu") (net 1))
-  (segment (start 179.25 56.245) (end 179.23 56.225) (width 0.4) (layer "F.Cu") (net 1))
   (segment (start 190.85 61.6) (end 190.85 62.65) (width 0.4) (layer "F.Cu") (net 1))
   (segment (start 178.27 53.3) (end 178.693 53.3) (width 0.4) (layer "F.Cu") (net 1))
@@
   (segment (start 174.90648 43.24952) (end 176.306 41.85) (width 0.4) (layer "F.Cu") (net 1))
   (segment (start 175.1 52.45) (end 175.1 47.832) (width 0.4) (layer "F.Cu") (net 1))
-  (segment (start 179.25 56.6) (end 179.25 56.245) (width 0.4) (layer "F.Cu") (net 1))
   (segment (start 177.673 52.703) (end 178.27 53.3) (width 0.4) (layer "F.Cu") (net 1))
   (segment (start 193.35 56.583573) (end 193.35 59.1) (width 0.4) (layer "F.Cu") (net 1))
@@
   (segment (start 194.953573 54.98) (end 193.35 56.583573) (width 0.4) (layer "F.Cu") (net 1))
   (segment (start 179.23 53.837) (end 178.693 53.3) (width 0.4) (layer "F.Cu") (net 1))
+  (segment (start 179.25 56.6) (end 179.25 56.245) (width 0.4) (layer "F.Cu") (net 1))
   (segment (start 195.27 54.96) (end 195.25 54.98) (width 0.4) (layer "F.Cu") (net 1))
+  (segment (start 179.25 56.245) (end 179.23 56.225) (width 0.4) (layer "F.Cu") (net 1))
   (segment (start 174.90648 46.20848) (end 174.90648 43.24952) (width 0.4) (layer "F.Cu") (net 1))
   (segment (start 174.3 56.7) (end 175.6 55.4) (width 0.4) (layer "F.Cu") (net 1))
@@
   (segment (start 191.574 54.98) (end 191.008 55.546) (width 0.25) (layer "F.Cu") (net 2))
   (segment (start 200.1 47.7) (end 200.1 60) (width 0.25) (layer "F.Cu") (net 2))
+  (segment (start 200.1 47.7) (end 199.375 47.7) (width 0.25) (layer "F.Cu") (net 2))
   (segment (start 180.5 65) (end 180.5 65.375) (width 0.4) (layer "F.Cu") (net 2))
   (segment (start 177.15 44.738) (end 176.306 43.894) (width 0.4) (layer "F.Cu") (net 2))
@@
   (segment (start 178.45448 46.04248) (end 176.306 43.894) (width 0.4) (layer "F.Cu") (net 2))
   (segment (start 195.27 43.595) (end 194 42.325) (width 0.4) (layer "F.Cu") (net 2))
+  (segment (start 200.1 60) (end 196.8 63.3) (width 0.25) (layer "F.Cu") (net 2))
+  (segment (start 196.8 63.3) (end 196.8 64.5) (width 0.25) (layer "F.Cu") (net 2))
+  (segment (start 199.375 47.7) (end 194 42.325) (width 0.25) (layer "F.Cu") (net 2))
   (segment (start 190.453 55.546) (end 189.85 56.149) (width 0.25) (layer "F.Cu") (net 2))
   (segment (start 194 53.73) (end 192.75 54.98) (width 0.25) (layer "F.Cu") (net 2))
@@
   (segment (start 186.433989 42.443393) (end 186.829107 42.838511) (width 0.25) (layer "B.Cu") (net 12))
   (segment (start 194.5 58.5) (end 192.325 58.5) (width 0.25) (layer "B.Cu") (net 12))
+  (segment (start 187.12 61.35) (end 187.0175 61.35) (width 0.25) (layer "B.Cu") (net 12))
   (segment (start 184.925489 51.979393) (end 184.925489 51.354511) (width 0.25) (layer "B.Cu") (net 12))
   (segment (start 189.64 61.35) (end 190.93 62.64) (width 0.25) (layer "B.Cu") (net 12))
@@
   (segment (start 187.06 49.22) (end 187.06 44.1) (width 0.25) (layer "B.Cu") (net 12))
   (segment (start 192.325 58.5) (end 191.516 59.309) (width 0.25) (layer "B.Cu") (net 12))
+  (segment (start 187.0175 61.35) (end 186.97 61.3975) (width 0.25) (layer "B.Cu") (net 12))
   (segment (start 197.49 70.68) (end 199.22 70.68) (width 0.25) (layer "B.Cu") (net 12))
   (segment (start 195.754 38.594) (end 195.754 38.1) (width 0.25) (layer "B.Cu") (net 12))
@@
   (segment (start 186.2225 68.07) (end 186.97 67.3225) (width 0.25) (layer "B.Cu") (net 13))
   (segment (start 182.17 68.07) (end 186.2225 68.07) (width 0.25) (layer "B.Cu") (net 13))
+  (segment (start 187.26 67.27) (end 187.0225 67.27) (width 0.4) (layer "B.Cu") (net 13))
+  (segment (start 187.0225 67.27) (end 186.97 67.3225) (width 0.4) (layer "B.Cu") (net 13))
   (segment (start 196.54 51.475) (end 196.54 54.175) (width 0.4) (layer "F.Cu") (net 14))
   (segment (start 194.15 61.6) (end 194.15 63.5) (width 0.4) (layer "F.Cu") (net 14))
