File: torque_motor_design_rp_shield.kicad_sch (KiCad schematic)
At the start: 34 parts, among them U1 ATtiny85-20S, U2 OPAMP, U3 OPAMP, U4 L78L05_SO8

Commit message: Add:Version_1
Parts:
- removed C1, C10, C12, C2, C3, C4, C6, C9: 10uF, Capacitor_Tantalum_SMD:CP_EIA-3216-18_Kemet-A, symbol Device:C_Polarized
- removed U4: L78L05_SO8, Package_TO_SOT_SMD:SOT-89-3, symbol Regulator_Linear:L78L05_SO8
- added C1, C10, C2, C4, C6, C9: 10uF, Capacitor_SMD:C_1206_3216Metric, symbol Device:C
- added C3: 100uF, Capacitor_SMD:CP_Elec_6.3x5.7, symbol Device:C
- added D2: zener, Diode_SMD:D_TUMD2, symbol Device:D_Zener
- added R4: 150, Resistor_SMD:R_0603_1608Metric, symbol Device:R
- C11, C5, C7, C8: footprint Capacitor_Tantalum_SMD:CP_EIA-3216-18_Kemet-A -> Capacitor_SMD:C_0201_0603Metric
- R1: value 49k -> 100k
- R3: footprint Resistor_SMD:R_2512_6332Metric -> Resistor_SMD:R_1206_3216Metric
- RV1: footprint Potentiometer_SMD:Potentiometer_Bourns_3224W_Vertical -> Potentiometer_SMD:Potentiometer_Bourns_3214W_Vertical
Connections:
- net +V: now also D6.2 (A), C1.1, C10.1, C6.1, R4.1; no longer D6.1 (K)
- net -V: now also D7.1 (K), C2.2, C4.1, C9.1; no longer D7.2 (A)
- net GND: now also C1.2, C10.2, C2.1, C3.2, C4.2, C6.2, C9.2, D2.2 (A); no longer D6.2 (A), D7.1 (K)
- net VCC_MCU_5V: now also C3.1, D2.1 (K), R4.2
- net at D1.2 (A), D5.1 (K), Motor+1.1 (Pin_1)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: now also D6.1 (K), D7.2 (A)
- no-connect marks 0 -> 2
Other:
- moved on the sheet: D6, D7
